File: br-project-template.kicad_pro/br-project-template.kicad_pro.kicad_pcb (KiCad board)
At the start: 2 copper layers, 34.1 x 44.1 mm, 33 parts, among them J3 DF13-4P-1.25V(21), J4 LABEL, U1 PCA9306D,118, U1 PCA9306DC1, U2 MIC5365-3.3YC5

Commit message: finish pcb (mostly)
Routing:
- net GND: vias 17 -> 20
Changed lines of the file:
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@@
 		)
 	)
-	(gr_text_box "PCBA:\n\n* PCBA Type: Standard\n* Assembly Side: Both Sides\n* Edge Rails/Fiducials: Added by JLCPCB\n* Confirm Parts Placement: Yes\n* Parts Selection: By Customer"
+	(gr_text_box "PCBA:\n\n* PCBA Type: Standard\n* Assembly Side: Top Side\n* Edge Rails/Fiducials: Added by JLCPCB\n* Confirm Parts Placement: Yes\n* Parts Selection: By Customer"
 		(start 90.49 137.72)
 		(end 162.29 157.72)
@@
 	)
 	(via
+		(at 197.06 117.27)
+		(size 0.6)
+		(drill 0.3)
+		(layers "F.Cu" "B.Cu")
+		(free yes)
+		(net 4)
+	)
+	(via
+		(at 204.7 119.39)
+		(size 0.6)
+		(drill 0.3)
+		(layers "F.Cu" "B.Cu")
+		(free yes)
+		(net 4)
+	)
+	(via
 		(at 203.0095 145.9611)
 		(size 0.9064)
@@
 	)
 	(via
+		(at 199.52 119.54)
+		(size 0.6)
+		(drill 0.3)
+		(layers "F.Cu" "B.Cu")
+		(free yes)
+		(net 4)
+	)
+	(via
 		(at 210.84 121.1)
 		(size 0.6)
@@
 	)
 	(zone
+		(net 4)
+		(net_name "GND")
+		(layer "F.Cu")
+		(hatch edge 0.5)
+		(priority 2)
+		(connect_pads
+			(clearance 0.5)
+		)
+		(min_thickness 0.25)
+		(filled_areas_thickness no)
+		(fill yes
+			(thermal_gap 0.5)
+			(thermal_bridge_width 0.5)
+		)
+		(polygon
+			(pts
+				(xy 195.18 116.63) (xy 196.5 115.35) (xy 197.9 115.35) (xy 200.76 118.99) (xy 202.19 119.62) (xy 202.64 116.94)
+				(xy 207.15 117.1) (xy 207.24 121.12) (xy 203.97 121.45) (xy 202.23 120.85) (xy 198.45 120.77) (xy 194.47 116.59)
+				(xy 195.16 116.62)
+			)
+		)
+	)
+	(zone
